Commit message: fixed issue with mtm model parsing

File: model/mtm.urdf.xacro (robot description, xacro)
@@ -172,7 +172,8 @@
     <transmission name="tran1" >
       <type>transmission_interface/SimpleTransmission</type>
-      <joint name="outer_yaw"/>
+      <joint name="outer_yaw">
+	<hardwareInterface>EffortJointInterface</hardwareInterface>
+      </joint>
       <actuator name="motor1">
-        <hardwareInterface>EffortJointInterface</hardwareInterface>
         <mechanicalReduction>1</mechanicalReduction>
       </actuator>
@@ -180,7 +181,8 @@
     <transmission name="tran2">
       <type>transmission_interface/SimpleTransmission</type>
-      <joint name="shoulder_pitch"/>
+      <joint name="shoulder_pitch">
+	<hardwareInterface>EffortJointInterface</hardwareInterface>
+      </joint>
       <actuator name="motor2">
-        <hardwareInterface>EffortJointInterface</hardwareInterface>
         <mechanicalReduction>1</mechanicalReduction>
       </actuator>
@@ -188,7 +190,8 @@
     <transmission name="tran3">
       <type>transmission_interface/SimpleTransmission</type>
-      <joint name="elbow_pitch"/>
+      <joint name="elbow_pitch">
+        <hardwareInterface>EffortJointInterface</hardwareInterface>
+	</joint>
       <actuator name="motor3">
-        <hardwareInterface>EffortJointInterface</hardwareInterface>
         <mechanicalReduction>1</mechanicalReduction>
       </actuator>
@@ -330,7 +333,8 @@
     <transmission name="tran4" type="transmission_interface/SimpleTransmission">
       <type>transmission_interface/SimpleTransmission</type>
-      <joint name="wrist_platform"/>
+      <joint name="wrist_platform">
+	<hardwareInterface>EffortJointInterface</hardwareInterface>
+	</joint>
       <actuator name="motor4">
-        <hardwareInterface>EffortJointInterface</hardwareInterface>
         <mechanicalReduction>1</mechanicalReduction>
       </actuator>
@@ -338,7 +342,8 @@
     <transmission name="tran5" type="transmission_interface/SimpleTransmission">
       <type>transmission_interface/SimpleTransmission</type>
-      <joint name="wrist_pitch"/>
+      <joint name="wrist_pitch">
+        <hardwareInterface>EffortJointInterface</hardwareInterface>
+	</joint>
       <actuator name="motor5">
-        <hardwareInterface>EffortJointInterface</hardwareInterface>
         <mechanicalReduction>1</mechanicalReduction>
       </actuator>
@@ -346,7 +351,8 @@
     <transmission name="tran6" type="transmission_interface/SimpleTransmission">
       <type>transmission_interface/SimpleTransmission</type>
-      <joint name="wrist_yaw"/>
+      <joint name="wrist_yaw">
+        <hardwareInterface>EffortJointInterface</hardwareInterface>
+	</joint>
       <actuator name="motor6">
-        <hardwareInterface>EffortJointInterface</hardwareInterface>
         <mechanicalReduction>1</mechanicalReduction>
       </actuator>
@@ -354,7 +360,8 @@
     <transmission name="tran7" type="transmission_interface/SimpleTransmission">
       <type>transmission_interface/SimpleTransmission</type>
-      <joint name="wrist_roll"/>
+      <joint name="wrist_roll">
+        <hardwareInterface>EffortJointInterface</hardwareInterface>
+	</joint>
       <actuator name="motor7">
-        <hardwareInterface>EffortJointInterface</hardwareInterface>
         <mechanicalReduction>1</mechanicalReduction>
       </actuator>
@@ -486,7 +493,8 @@
     <transmission name="tran4">
       <type>transmission_interface/SimpleTransmission</type>
-      <joint name="wrist_platform"/>
+      <joint name="wrist_platform">
+        <hardwareInterface>EffortJointInterface</hardwareInterface>
+	</joint>
       <actuator name="motor4">
-        <hardwareInterface>EffortJointInterface</hardwareInterface>
         <mechanicalReduction>1</mechanicalReduction>
       </actuator>
@@ -494,7 +502,8 @@
     <transmission name="tran5">
       <type>transmission_interface/SimpleTransmission</type>
-      <joint name="wrist_pitch"/>
+      <joint name="wrist_pitch">
+        <hardwareInterface>EffortJointInterface</hardwareInterface>
+	</joint>
       <actuator name="motor5">
-        <hardwareInterface>EffortJointInterface</hardwareInterface>
         <mechanicalReduction>1</mechanicalReduction>
       </actuator>
@@ -502,7 +511,8 @@
     <transmission name="tran6">
       <type>transmission_interface/SimpleTransmission</type>
-      <joint name="wrist_yaw"/>
+      <joint name="wrist_yaw">
+        <hardwareInterface>EffortJointInterface</hardwareInterface>
+	</joint>
       <actuator name="motor6">
-        <hardwareInterface>EffortJointInterface</hardwareInterface>
         <mechanicalReduction>1</mechanicalReduction>
       </actuator>
@@ -510,7 +520,8 @@
     <transmission name="tran7">
       <type>transmission_interface/SimpleTransmission</type>
-      <joint name="wrist_roll"/>
+      <joint name="wrist_roll">
+	<hardwareInterface>EffortJointInterface</hardwareInterface>
+      </joint>
       <actuator name="motor7">
-        <hardwareInterface>EffortJointInterface</hardwareInterface>
         <mechanicalReduction>1</mechanicalReduction>
       </actuator>
